File: usbpd/usbpd/usbpd.kicad_pcb (KiCad board)
At the start: 2 copper layers, 70 x 40 mm, 50 parts, among them J1 USB_C_Receptacle, J2 Conn_02x02_Top_Bottom, J3 Conn_02x05_Counter_Clockwise, J4 Conn_01x02_Male, U1 TPS565201DDC, U2 MCP73223-C2S, U3 FUSB302BMPX, U4 CP2102N-A02-GQFN20

Commit message: m
Parts:
- removed J4: Conn_01x02_Male, Connector_JST:JST_PH_B2B-PH-SM4-TB_1x02-1MP_P2.00mm_Vertical
- removed R2: 10K, Resistors:0603
- removed R9: 1K, Resistor_SMD:R_0603_1608Metric
- removed TP10, TP11, TP14, TP5, TP6, TP7, TP8, TP9: TestPoint, Connectors:PAD.03X.03
- added C19: NC, Capacitor_SMD:C_0603_1608Metric, F.Cu at (130.5, 96.8)
- added C20: whatever 500V 0805, Capacitor_SMD:C_0805_2012Metric, F.Cu at (113.2, 107.5)
- added C21: 200-600pF, Capacitor_SMD:C_0603_1608Metric, F.Cu at (226.1, 35.1)
- added C22: 200-600pF, Capacitor_SMD:C_0603_1608Metric, F.Cu at (235.3, 27.4)
- added C23: 100uF, Capacitor_SMD:C_Elec_8x10.2, F.Cu at (138.1, 75.2)
- added C24: 100uF, Capacitor_SMD:C_Elec_8x10.2, F.Cu at (138.0, 54.0)
- added C25: 10uF X5R/X7R 25V, Capacitor_SMD:C_0603_1608Metric, F.Cu at (130.5, 60.6)
- added C26: 10uF X5R/X7R 25V, Capacitor_SMD:C_0603_1608Metric, F.Cu at (133.1, 60.6)
- added C27: 10uF X5R/X7R 25V, Capacitor_SMD:C_0603_1608Metric, F.Cu at (132.8, 57.0)
- added C28: 10uF X5R/X7R 25V, Capacitor_SMD:C_0603_1608Metric, F.Cu at (131.1, 57.0)
- added C29: 4.7uF, Capacitor_SMD:C_0603_1608Metric, F.Cu at (235.3, 29.9)
- added C30: 0.1uF, Capacitor_SMD:C_0603_1608Metric, F.Cu at (227.1, 37.7)
- added C31: 4.7uF, Capacitor_SMD:C_0603_1608Metric, F.Cu at (239.3, 27.4)
- added C32: 0.1uF, Capacitor_SMD:C_0603_1608Metric, F.Cu at (217.6, 48.6)
- added C33: 4.7uF, Capacitor_SMD:C_0603_1608Metric, F.Cu at (225.6, 40.7)
- added D1: SMF22VTR, Diode_SMD:D_SOD-123F, F.Cu at (144.2, 96.8)
- added D3: SMF22VTR, Diode_SMD:D_SOD-123F, F.Cu at (123.3, 99.0)
- added FB1: Ferrite_Bead, Inductor_SMD:L_0805_2012Metric, F.Cu at (121.8, 89.3)
- added FL1: 0603USB-251MLB, Inductor_SMD:L_CommonModeChoke_Coilcraft_0603USB, F.Cu at (127.3, 100.5)
- added FL2: 0603USB-251MLB, Inductor_SMD:L_CommonModeChoke_Coilcraft_0603USB, F.Cu at (247.3, 18.4)
- added FL3: LCV70-701-2PL-TL00, aep:ACM70V, F.Cu at (138.1, 96.8)
- added J5: USB_C_Receptacle, lib:USB-C-DX07S, F.Cu at (121.5, 105.2)
- added L3: INDUCTOR, Inductor_SMD:L_1206_3216Metric, F.Cu at (127.1, 73.2)
- added L7: INDUCTOR, Inductor_SMD:L_1206_3216Metric, F.Cu at (127.7, 56.9)
- added Q1: STL6P3LLH6, lib:TRANS_STL6P3LLH6, F.Cu at (127.3, 80.7)
- added R10: 0, Resistor_SMD:R_0603_1608Metric, F.Cu at (123.5, 85.3)
- added R11: NC, Resistor_SMD:R_0603_1608Metric, F.Cu at (115.1, 107.7)
- added R12: 1K, Resistor_SMD:R_0603_1608Metric, F.Cu at (157.4, 78.5)
- added R13: 10K, Resistor_SMD:R_0603_1608Metric, F.Cu at (125.9, 62.9)
- added R14: 2.49K, Resistor_SMD:R_0603_1608Metric, F.Cu at (127.7, 64.5)
- added R16: 22.1K, Resistor_SMD:R_0603_1608Metric, F.Cu at (231.1, 38.6)
- added R17: 47.5K, Resistor_SMD:R_0603_1608Metric, F.Cu at (221.6, 48.6)
- added R18: 0, Resistor_SMD:R_0603_1608Metric, F.Cu at (235.1, 34.9)
- added R19: 0, Resistor_SMD:R_0603_1608Metric, F.Cu at (238.5, 32.4)
- added R20: 1K, Resistor_SMD:R_0603_1608Metric, F.Cu at (217.6, 53.6)
- added R21: 0, Resistor_SMD:R_0603_1608Metric, F.Cu at (225.6, 45.7)
- added R22: 0, Resistor_SMD:R_0603_1608Metric, F.Cu at (128.9, 96.8)
- added U5: CP2102N-A01-GQFN24, Package_DFN_QFN:QFN-24-1EP_4x4mm_P0.5mm_EP2.6x2.6mm, F.Cu at (129.9, 29.6)
- C1: value 100uF 50V -> NC; footprint Capacitor_SMD:CP_Elec_6.3x7.7 -> Capacitor_SMD:C_0603_1608Metric
- C10: value 100nF 50V -> 10uF X5R/X7R 25V; footprint Capacitors:0603 -> Capacitor_SMD:C_0603_1608Metric
- C11, C12: value 200-600pF -> 10uF X5R/X7R 25V
- C14, C16: value 0.1uF -> 1uF
- C15, C17: value 4.7uF -> NC
- C18: value 0.1uF -> NC
- C2: value 0.1uF 20V -> 1uF; footprint Capacitors:0603 -> Capacitor_SMD:C_0603_1608Metric
- C3: value 10uF 20V -> 10uF X5R/X7R 25V; footprint Capacitors:0805 -> Capacitor_SMD:C_0603_1608Metric
- C4: value 10uF 20V -> NC; footprint Capacitors:0805 -> Capacitor_SMD:C_0603_1608Metric
- C5: value 100nF 50V -> NC; footprint Capacitors:0603 -> Capacitor_SMD:C_0603_1608Metric
- C6, C7: value 4.7uF 50V -> 1uF; footprint Capacitors:0603 -> Capacitor_SMD:C_0603_1608Metric
- C8, C9: value 22uF -> 200-600pF; footprint Capacitors:0805 -> Capacitor_SMD:C_0603_1608Metric
- J2: value Conn_02x02_Top_Bottom -> Conn_02x06_Odd_Even; footprint Connector_Molex:Molex_Micro-Fit_3.0_43045-0400_2x02_P3.00mm_Horizontal -> Connector_PinHeader_2.54mm:PinHeader_2x06_P2.54mm_Vertical_SMD
- J3: footprint Connector_PinHeader_2.54mm:PinHeader_2x05_P2.54mm_Vertical -> Connector_PinHeader_2.54mm:PinHeader_2x05_P2.54mm_Vertical_SMD
- L1: value 4.7uH -> NR6045T100M; footprint Inductor_SMD:L_Coilcraft_XxL4020 -> Inductor_SMD:L_Taiyo-Yuden_NR-60xx
- R1: value 54K9 -> NC; footprint Resistors:0603 -> Resistor_SMD:R_0603_1608Metric
- R3, R4: footprint Resistors:0603 -> Resistor_SMD:R_0603_1608Metric
- R5: value 22K -> 1K; footprint Resistors:0603 -> Resistor_SMD:R_0603_1608Metric
- R6: value 5K -> 1K; footprint Resistors:0603 -> Resistor_SMD:R_0603_1608Metric
- R7: value 22.1K -> NC
- R8: value 47.5K -> 0
- TP1, TP2: footprint Connectors:PAD.03X.03 -> digikey-footprints:Test-Point-Pin_Drill2.79mm
- TP3, TP4: footprint Connectors:PAD.03X.03 -> TestPoint:TestPoint_Pad_D1.5mm
- U1: value TPS565201DDC -> TPD4E02B04DQA; footprint Package_TO_SOT_SMD:SOT-23-6 -> aep:USON-10_2.5x1.0mm_P0.5mm_HAXED_MIDDLE
- U2: value MCP73223-C2S -> STUSB4500QTR; footprint Package_DFN_QFN:DFN-10-1EP_3x3mm_P0.5mm_EP1.55x2.48mm -> Package_DFN_QFN:QFN-24-1EP_4x4mm_P0.5mm_EP2.7x2.7mm
- U3: value FUSB302BMPX -> TPD4E02B04DQA; footprint Package_DFN_QFN:WQFN-14-1EP_2.5x2.5mm_P0.5mm_EP1.45x1.45mm -> aep:USON-10_2.5x1.0mm_P0.5mm_HAXED_MIDDLE
- U4: value CP2102N-A02-GQFN20 -> TPSM53602; footprint lib:IC_CP2102N-A01-GQFN20 -> aep:B3QFN
- moved TP3 138.5 mm to (125.7, 67.2)
- moved TP2 138.2 mm to (114.9, 69.0)
- moved C12 138.1 mm to (130.5, 68.8)
- moved C11 135.8 mm to (133.1, 68.8), turned to 180 degrees
- moved U3 128.2 mm to (132.4, 101.5)
- moved L1 127.3 mm to (122.0, 94.2), turned to 180 degrees
- moved TP4 127.3 mm to (137.4, 63.2)
- moved TP1 126.7 mm to (114.9, 62.0)
- moved C2 126.4 mm to (121.9, 87.0), turned to 180 degrees
- moved J2 126.2 mm to (118.9, 32.5), turned to 90 degrees
- moved R1 125.7 mm to (123.5, 83.5), turned to 180 degrees
- moved U4 124.4 mm to (131.8, 64.8), turned to 180 degrees
- moved R8 124.0 mm to (136.6, 66.5), turned to 90 degrees
- moved C10 122.9 mm to (132.6, 71.8), turned to 270 degrees
- moved C1 121.5 mm to (120.3, 83.5), turned to 180 degrees
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Connections:
- C1 pad 1: VBAT -> Net-(C1-Pad1)
- C10 pad 1: GND -> VBUSOK
- C10 pad 2: 5V -> GND
- C11 pad 1: CC1 -> VBUSOK
- C12 pad 1: CC2 -> VBUSOK
- C13 pad 1: Net-(C13-Pad1) -> GND
- C13 pad 2: GND -> Net-(C13-Pad2)
- C14 pad 1: Net-(C13-Pad1) -> VBUSOK
- C14 pad 2: GND -> Net-(C14-Pad2)
- C15 pad 1: 5V -> Net-(C15-Pad1)
- C16 pad 1: 5V -> GND
- C16 pad 2: GND -> Net-(C16-Pad2)
- C18 pad 1: Net-(C17-Pad1) -> Net-(C18-Pad1)
- C2 pad 1: GND -> Net-(C2-Pad1)
- C2 pad 2: VBAT -> GND
- C3 pad 1: GND -> VBUSOK
- C3 pad 2: VBAT -> GND
- C4 pad 1: GND -> Net-(C4-Pad1)
- C4 pad 2: VBAT -> GND
- C5 pad 2: Net-(C5-Pad2) -> GND
- C6 pad 1: GND -> VBUS
- C6 pad 2: VBUS -> GND
- C7 pad 2: VBAT -> Net-(C7-Pad2)
- C8 pad 1: GND -> CC2
- C8 pad 2: 5V -> GND
- C9 pad 1: GND -> CC1
- C9 pad 2: 5V -> GND
- J1 pad A1: GND -> /S1
- J1 pad A12: GND -> /S1
- J1 pad A4: VBUS -> Net-(D1-Pad1)
- J1 pad A9: VBUS -> Net-(D1-Pad1)
- J1 pad B1: GND -> /S1
- J1 pad B12: GND -> /S1
- J1 pad B4: VBUS -> Net-(D1-Pad1)
- J1 pad B9: VBUS -> Net-(D1-Pad1)
- J1 pad S1: GND -> /S1
- J2 pad 1: 5V -> Net-(J2-Pad1)
- J2 pad 2: (no net) -> Net-(J2-Pad2)
- J2 pad 3: (no net) -> Net-(J2-Pad3)
- J2 pad 4: (no net) -> Net-(J2-Pad4)
- J3 pad 5: INT -> (no net)
- J3 pad 6: TXD -> (no net)
- J3 pad 7: RXD -> (no net)
- J3 pad 8: RTS -> (no net)
- J3 pad 9: CTS -> (no net)
- L1 pad 1: Net-(C5-Pad2) -> Net-(C2-Pad1)
- L1 pad 2: 5V -> Net-(D3-Pad1)
- R1 pad 1: 5V -> VBUS
- R1 pad 2: Net-(R1-Pad2) -> Net-(C1-Pad1)
- R3 pad 1: Net-(R3-Pad1) -> VBUS
- R3 pad 2: GND -> Net-(R3-Pad2)
- R4 pad 1: Net-(R4-Pad1) -> VBUSOK
- R4 pad 2: (no net) -> Net-(R4-Pad2)
- R5 pad 1: VBAT -> Net-(Q1-Pad4)
- R5 pad 2: BAT_SENSE -> VBUS
- R6 pad 1: BAT_SENSE -> Net-(R6-Pad1)
- R6 pad 2: GND -> Net-(Q1-Pad4)
- R7 pad 2: Net-(R7-Pad2) -> Net-(C15-Pad1)
- R8 pad 1: Net-(R7-Pad2) -> VBUSOK
- R8 pad 2: GND -> Net-(R8-Pad2)
- U1 pad 1: GND -> CC2
- U1 pad 2: Net-(C5-Pad2) -> Net-(C5-Pad1)
- U1 pad 3: VBAT -> GND
- U1 pad 4: Net-(R1-Pad2) -> Net-(C4-Pad1)
- U1 pad 5: VBAT -> CC1
- U1 pad 6: Net-(C5-Pad1) -> CC1
- U2 pad 1: VBUS -> CC1
- U2 pad 10: Net-(R3-Pad1) -> GND
- U2 pad 11: GND -> (no net)
- U2 pad 2: VBUS -> CC1
- U2 pad 3: VBAT -> (no net)
- U2 pad 4: VBAT -> CC2
- U2 pad 5: (no net) -> CC2
- U2 pad 6: (no net) -> GND
- U2 pad 7: Net-(R4-Pad1) -> SCL
- U2 pad 8: GND -> SDA
- U2 pad 9: GND -> Net-(R4-Pad2)
- U3 pad 1: CC2 -> Net-(C17-Pad1)
- U3 pad 10: CC1 -> Net-(C17-Pad1)
- U3 pad 2: VBUS -> Net-(C18-Pad1)
- U3 pad 3: Net-(C13-Pad1) -> GND
- U3 pad 4: Net-(C13-Pad1) -> CC1
- U3 pad 5: INT -> CC2
- U3 pad 6: SCL -> CC2
- U3 pad 7: SDA -> CC1
- U3 pad 9: GND -> Net-(C18-Pad1)
- U4 pad 1: (no net) -> VBUSOK
- U4 pad 10: (no net) -> GND
- U4 pad 11: (no net) -> GND
- U4 pad 12: GND -> (no net)
- U4 pad 13: (no net) -> Net-(TP3-Pad1)
- U4 pad 14: (no net) -> VBUSOK
- U4 pad 15: CTS -> GND
- U4 pad 2: (no net) -> Net-(R8-Pad2)
- U4 pad 4: D+ -> (no net)
- U4 pad 5: D- -> (no net)
- U4 pad 6: Net-(C17-Pad1) -> Net-(TP4-Pad1)
- U4 pad 8: Net-(R7-Pad2) -> 5V
Routing:
- net /S1: track 0.00 -> 51.7 mm
- net VBUSOK: track 0.00 -> 46.2 mm
- net Net-(D3-Pad1): track 0.00 -> 45.9 mm, vias 0 -> 4
- net VBUS: track 0.00 -> 37.3 mm
- net 5V: track 0.00 -> 36.3 mm
- net Net-(D1-Pad1): track 0.00 -> 29.8 mm, vias 0 -> 4
- net D-: track 0.00 -> 28.5 mm, vias 0 -> 2
- net D+: track 0.00 -> 26.3 mm, vias 0 -> 4
- net CC1: track 0.00 -> 24.2 mm, vias 0 -> 3
- net Net-(C20-Pad1): track 0.00 -> 23.8 mm
- net CC2: track 0.00 -> 23.5 mm, vias 0 -> 2
- net GND: track 0.00 -> 15.0 mm, vias 0 -> 22
- net Net-(C2-Pad1): track 0.00 -> 9.55 mm
- net Net-(C16-Pad2): track 0.00 -> 6.57 mm
- net Net-(TP3-Pad1): track 0.00 -> 4.26 mm
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- added copper zone on F.Cu, net 5V
- added copper zone on B.Cu, net GND
- added copper zone on F.Cu, net GND
- added copper zone on F.Cu, net VBUSOK
Other:
- board size 70 x 40 mm -> 70 x 84 mm
- net class Default: trace_width 0.25 -> 0.2; via_dia 0.8 -> 0.4; via_drill 0.4 -> 0.2
- rule via_min_drill: 0.3 -> 0.2
- rule via_min_size: 0.4 -> 0.25
- board text added: "5V"
- board text added: "GND"
- board text added: "VBUS"
- board text added: "VBUSok"

Commit message: m
Parts:
- removed C22: 200-600pF, Capacitor_SMD:C_0603_1608Metric
- removed FL2: 0603USB-251MLB, Inductor_SMD:L_CommonModeChoke_Coilcraft_0603USB
- removed TP3, TP4: TestPoint, TestPoint:TestPoint_Pad_D1.5mm
- added D10: LED, digikey-footprints:LED_0603, F.Cu at (142.1, 65.5)
- added D2: LED, digikey-footprints:LED_0603, F.Cu at (167.3, 105.7)
- added D4: LED, digikey-footprints:LED_0603, F.Cu at (169.1, 105.8)
- added D5: LED, digikey-footprints:LED_0603, F.Cu at (174.3, 105.8)
- added D6: LED, digikey-footprints:LED_0603, F.Cu at (165.7, 105.8)
- added D7: LED, digikey-footprints:LED_0603, F.Cu at (172.6, 105.8)
- added D8: LED, digikey-footprints:LED_0603, F.Cu at (170.8, 105.8)
- added D9: LED, digikey-footprints:LED_0603, F.Cu at (176.1, 105.7)
- added J10: Conn_01x04_Female, aep:Castellated_Edge_1x4_P2.54mm, F.Cu at (110.0, 74.9)
- added J11: Conn_01x04_Female, aep:Castellated_Edge_1x4_P2.54mm, F.Cu at (110.0, 95.2)
- added J12: Conn_01x04_Female, aep:Castellated_Edge_1x4_P2.54mm, F.Cu at (110.0, 85.1)
- added J13: Conn_01x06, Connector:Tag-Connect_TC2030-IDC-FP_2x03_P1.27mm_Vertical, F.Cu at (169.2, 59.2)
- added J4: Conn_01x04_Female, aep:Castellated_Edge_1x4_P2.54mm, F.Cu at (180.0, 100.3)
- added J6: Conn_01x04_Female, aep:Castellated_Edge_1x4_P2.54mm, F.Cu at (180.0, 69.8)
- added J7: Conn_01x04_Female, aep:Castellated_Edge_1x4_P2.54mm, F.Cu at (180.0, 90.2)
- added J8: Conn_01x04_Female, aep:Castellated_Edge_1x4_P2.54mm, F.Cu at (180.0, 80.0)
- added J9: Conn_01x04_Female, aep:Castellated_Edge_1x4_P2.54mm, F.Cu at (110.0, 64.8)
- added R15: 1K, Resistor_SMD:R_0603_1608Metric, F.Cu at (165.7, 102.5)
- added R2: 1K, Resistor_SMD:R_0603_1608Metric, F.Cu at (167.3, 102.5)
- added R23: 1K, Resistor_SMD:R_0603_1608Metric, F.Cu at (170.8, 102.5)
- added R24: 1K, Resistor_SMD:R_0603_1608Metric, F.Cu at (176.0, 102.5)
- added R25: 1K, Resistor_SMD:R_0603_1608Metric, F.Cu at (139.7, 64.7)
- added R26: 100K, Resistor_SMD:R_0603_1608Metric, F.Cu at (139.7, 66.3)
- added R27: 1K, Resistor_SMD:R_0603_1608Metric, F.Cu at (160.5, 66.5)
- added R9: 1K, Resistor_SMD:R_0603_1608Metric, F.Cu at (174.3, 102.5)
- added U6: AZ1117CH-3_3TRG1, digikey-footprints:SOT-223, F.Cu at (156.0, 58.5)
- C15, C17, C18: value NC -> 10uF
- C21: value 200-600pF -> 10uF
- R22: value 0 -> 1K
- R7: value NC -> 1K
- U3: value TPD4E02B04DQA -> STM32F070F6Px; footprint aep:USON-10_2.5x1.0mm_P0.5mm_HAXED_MIDDLE -> Package_SO:TSSOP-20_4.4x6.5mm_P0.65mm
- moved C8 122.6 mm to (141.4, 93.0), turned to 90 degrees
- moved C4 104.3 mm to (157.2, 88.6), turned to 180 degrees
- moved R19 96.4 mm to (160.2, 88.6), turned to 180 degrees
- moved C9 96.3 mm to (139.9, 92.2), turned to 90 degrees
- moved C31 95.5 mm to (165.8, 88.2), turned to 270 degrees
- moved R18 93.1 mm to (160.2, 90.2), turned to 180 degrees
- moved C29 92.2 mm to (169.4, 94.4), turned to 180 degrees
- moved C7 88.1 mm to (145.8, 88.0), turned to 270 degrees
- moved R3 87.8 mm to (141.2, 88.0), turned to 90 degrees
- moved C5 86.1 mm to (157.2, 90.2), turned to 180 degrees
- moved C6 84.0 mm to (142.8, 88.0), turned to 90 degrees
- moved R16 82.1 mm to (169.4, 92.8)
- moved C30 82.1 mm to (169.4, 96.0), turned to 180 degrees
- moved R7 82.0 mm to (169.1, 102.5), turned to 90 degrees
- moved C18 80.6 mm to (162.5, 59.5)
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Connections:
- C15 pad 1: Net-(C15-Pad1) -> 5V
- C16 pad 2: Net-(C16-Pad2) -> VBUS
- C17 pad 1: Net-(C17-Pad1) -> 3.3V
- C18 pad 1: Net-(C18-Pad1) -> 3.3V
- C19 pad 1: Net-(C16-Pad2) -> VBUS
- C21 pad 1: CC1 -> 3.3V
- C4 pad 1: Net-(C4-Pad1) -> D+
- C5 pad 1: Net-(C5-Pad1) -> D-
- D1 pad 1: Net-(D1-Pad1) -> /VIN
- FL1 pad 1: Net-(C4-Pad1) -> IN_D+
- FL1 pad 2: D+ -> D-
- FL1 pad 3: Net-(C5-Pad1) -> D+
- FL1 pad 4: D- -> IN_D-
- FL3 pad 1: /S1 -> /VIN
- FL3 pad 2: Net-(D1-Pad1) -> /S1
- FL3 pad 3: Net-(C16-Pad2) -> GND
- FL3 pad 4: GND -> VBUS
- J1 pad A4: Net-(D1-Pad1) -> /VIN
- J1 pad A6: D- -> IN_D-
- J1 pad A7: D+ -> IN_D+
- J1 pad A9: Net-(D1-Pad1) -> /VIN
- J1 pad B4: Net-(D1-Pad1) -> /VIN
- J1 pad B6: D- -> IN_D-
- J1 pad B7: D+ -> IN_D+
- J1 pad B9: Net-(D1-Pad1) -> /VIN
- J2 pad 1: Net-(J2-Pad1) -> USART_DTR
- J2 pad 4: Net-(J2-Pad4) -> USART_TX
- J2 pad 6: Net-(J2-Pad6) -> USART_RX
- J2 pad 8: Net-(J2-Pad8) -> USART_RTS
- J3 pad 1: (no net) -> STUSB_VSYS
- J3 pad 2: (no net) -> ALERT
- J3 pad 3: SDA -> A_B_SIDE
- J3 pad 4: SCL -> SDA
- J3 pad 5: (no net) -> SCL
- J3 pad 6: (no net) -> POER_OK3
- J3 pad 7: (no net) -> POER_OK2
- J3 pad 8: (no net) -> ATTACH
- J5 pad A6: D- -> IN_D-
- J5 pad A7: D+ -> IN_D+
- J5 pad B6: D- -> IN_D-
- J5 pad B7: D+ -> IN_D+
- R22 pad 1: Net-(C16-Pad2) -> Net-(D7-Pad1)
- R22 pad 2: VBUS -> ALERT
- R7 pad 1: VBUS -> Net-(D4-Pad1)
- R7 pad 2: Net-(C15-Pad1) -> POER_OK2
- U1 pad 2: Net-(C5-Pad1) -> IN_D+
- U1 pad 3: GND -> /S1
- U1 pad 4: Net-(C4-Pad1) -> IN_D-
- U1 pad 7: Net-(C4-Pad1) -> IN_D-
- U1 pad 8: GND -> /S1
- U1 pad 9: Net-(C5-Pad1) -> IN_D+
- U2 pad 11: (no net) -> ATTACH
- U2 pad 14: (no net) -> POER_OK3
- U2 pad 17: (no net) -> A_B_SIDE
- U2 pad 19: (no net) -> ALERT
- U2 pad 20: (no net) -> POER_OK2
- U2 pad 22: (no net) -> STUSB_VSYS
- U3 pad 1: Net-(C17-Pad1) -> Net-(R27-Pad1)
- U3 pad 10: Net-(C17-Pad1) -> USART_DTR
- U3 pad 2: Net-(C18-Pad1) -> (no net)
- U3 pad 3: GND -> (no net)
- U3 pad 4: CC1 -> USART_RESET
- U3 pad 5: CC2 -> 3.3V
- U3 pad 6: CC2 -> (no net)
- U3 pad 7: CC1 -> USART_RTS
- U3 pad 8: GND -> USART_TX
- U3 pad 9: Net-(C18-Pad1) -> USART_RX
- U4 pad 12: (no net) -> GND
- U5 pad 19: Net-(J2-Pad8) -> USART_RTS
- U5 pad 20: Net-(J2-Pad6) -> USART_RX
- U5 pad 21: Net-(J2-Pad4) -> USART_TX
- U5 pad 23: Net-(J2-Pad1) -> USART_DTR
Routing:
- net 5V: track 36.3 -> 160.5 mm
- net POER_OK2: track 0.00 -> 51.7 mm, vias 0 -> 3
- net STUSB_VSYS: track 0.00 -> 48.9 mm, vias 0 -> 2
- net ATTACH: track 0.00 -> 46.8 mm, vias 0 -> 3
- net ALERT: track 0.00 -> 46.1 mm, vias 0 -> 3
- net 3.3V: track 0.00 -> 45.8 mm
- net POER_OK3: track 0.00 -> 43.7 mm, vias 0 -> 3
- net A_B_SIDE: track 0.00 -> 42.0 mm, vias 0 -> 2
- net USART_TX: track 0.00 -> 41.3 mm, vias 0 -> 2
- net IN_D+: track 0.00 -> 39.8 mm, vias 0 -> 5
- net USART_DTR: track 0.00 -> 39.5 mm, vias 0 -> 2
- net USART_RTS: track 0.00 -> 39.4 mm, vias 0 -> 2
- net IN_D-: track 0.00 -> 38.6 mm, vias 0 -> 3
- net USART_RX: track 0.00 -> 36.1 mm, vias 0 -> 2
- net Net-(J2-Pad3): track 0.00 -> 30.1 mm
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- added copper zone on F.Cu, net (none)
- added copper zone on B.Cu, net /S1
- added copper zone on F.Cu, net /S1
- added copper zone on B.Cu, net /VIN
- added copper zone on F.Cu, net /VIN
- added copper zone on F.Cu, net VBUS
Other:
- board size 70 x 84 mm -> 70 x 57 mm
- board text added: "USB-JUZZZZZ v1"
