File: usbpd/usbpd/usbpd.sch (KiCad schematic (older format))
At the start: 50 parts, among them J1 USB_C_Receptacle, J2 Conn_02x02_Top_Bottom, J3 Conn_02x05_Counter_Clockwise, J4 Conn_01x02_Male, U1 TPS565201DDC, U2 MCP73223-C2S, U3 FUSB302BMPX, U4 CP2102N-A02-GQFN20

Commit message: m
Parts:
- removed C1: 100uF 50V, Capacitor_SMD:CP_Elec_6.3x7.7, symbol Device:CP
- removed J2: Conn_02x02_Top_Bottom, Connector_Molex:Molex_Micro-Fit_3.0_43045-0400_2x02_P3.00mm_Horizontal, symbol Connector_Generic:Conn_02x02_Top_Bottom
- removed J4: Conn_01x02_Male, Connector_JST:JST_PH_B2B-PH-SM4-TB_1x02-1MP_P2.00mm_Vertical, symbol Connector:Conn_01x02_Male
- removed L1: 4.7uH, Inductor_SMD:L_Coilcraft_XxL4020, symbol Device:L
- removed R2: 10K, Resistors:0603, symbol Device:R
- removed R9: 1K, Resistor_SMD:R_0603_1608Metric, symbol Device:R
- removed TP10, TP11, TP14, TP5, TP6, TP7, TP8, TP9: TestPoint, Connectors:PAD.03X.03, symbol Connector:TestPoint
- removed U1: TPS565201DDC, Package_TO_SOT_SMD:SOT-23-6, symbol Regulator_Switching:TPS565208
- removed U2: MCP73223-C2S, Package_DFN_QFN:DFN-10-1EP_3x3mm_P0.5mm_EP1.55x2.48mm, symbol aep:MCP73223
- removed U3: FUSB302BMPX, Package_DFN_QFN:WQFN-14-1EP_2.5x2.5mm_P0.5mm_EP1.45x1.45mm, symbol Interface_USB:FUSB302BMPX
- removed U4: CP2102N-A02-GQFN20, lib:IC_CP2102N-A01-GQFN20, symbol aep:CP2102N-A02-GQFN20
- added C1, C19: NC, Capacitor_SMD:C_0603_1608Metric, symbol Device:C
- added C20: whatever 500V 0805, Capacitor_SMD:C_0805_2012Metric, symbol Device:C
- added C21, C22: 200-600pF, Capacitor_SMD:C_0603_1608Metric, symbol Device:C
- added C23, C24: 100uF, Capacitor_SMD:C_Elec_8x10.2, symbol Device:CP
- added C25, C26, C27, C28: 10uF X5R/X7R 25V, Capacitor_SMD:C_0603_1608Metric, symbol Device:C
- added C29, C31, C33: 4.7uF, Capacitor_SMD:C_0603_1608Metric, symbol Device:C
- added C30, C32: 0.1uF, Capacitor_SMD:C_0603_1608Metric, symbol Device:C
- added D1, D3: SMF22VTR, Diode_SMD:D_SOD-123F, symbol Device:D_Schottky
- added FB1: Ferrite_Bead, Inductor_SMD:L_0805_2012Metric, symbol Device:Ferrite_Bead
- added FL1, FL2: 0603USB-251MLB, Inductor_SMD:L_CommonModeChoke_Coilcraft_0603USB, symbol Device:EMI_Filter_CommonMode
- added FL3: LCV70-701-2PL-TL00, aep:ACM70V, symbol Device:EMI_Filter_LL_1423
- added J2: Conn_02x06_Odd_Even, Connector_PinHeader_2.54mm:PinHeader_2x06_P2.54mm_Vertical_SMD, symbol Connector_Generic:Conn_02x06_Odd_Even
- added J5: USB_C_Receptacle, lib:USB-C-DX07S, symbol Connector:USB_C_Receptacle
- added L1: NR6045T100M, Inductor_SMD:L_Taiyo-Yuden_NR-60xx, symbol pspice:INDUCTOR
- added L3, L7: INDUCTOR, Inductor_SMD:L_1206_3216Metric, symbol pspice:INDUCTOR
- added Q1: STL6P3LLH6, TRANS_STL6P3LLH6, symbol STL6P3LLH6:STL6P3LLH6
- added R10, R18, R19, R21, R22: 0, Resistor_SMD:R_0603_1608Metric, symbol Device:R
- added R11: NC, Resistor_SMD:R_0603_1608Metric, symbol Device:R
- added R12, R20: 1K, Resistor_SMD:R_0603_1608Metric, symbol Device:R
- added R13: 10K, Resistor_SMD:R_0603_1608Metric, symbol Device:R
- added R14: 2.49K, Resistor_SMD:R_0603_1608Metric, symbol Device:R
- added R16: 22.1K, Resistor_SMD:R_0603_1608Metric, symbol Device:R
- added R17: 47.5K, Resistor_SMD:R_0603_1608Metric, symbol Device:R
- added U1, U3: TPD4E02B04DQA, aep:USON-10_2.5x1.0mm_P0.5mm_HAXED_MIDDLE, symbol aep:TPD4E02B04DQA
- added U2: STUSB4500QTR, Package_DFN_QFN:QFN-24-1EP_4x4mm_P0.5mm_EP2.7x2.7mm, symbol Interface_USB:STUSB4500QTR
- added U4: TPSM53602, aep:B3QFN, symbol aep:TPSM53602
- added U5: CP2102N-A01-GQFN24, Package_DFN_QFN:QFN-24-1EP_4x4mm_P0.5mm_EP2.6x2.6mm, symbol Interface_USB:CP2102N-A01-GQFN24
- C10: value 100nF 50V -> 10uF X5R/X7R 25V; footprint Capacitors:0603 -> Capacitor_SMD:C_0603_1608Metric
- C11, C12: value 200-600pF -> 10uF X5R/X7R 25V
- C14, C16: value 0.1uF -> 1uF
- C15, C17: value 4.7uF -> NC
- C18: value 0.1uF -> NC
- C2: value 0.1uF 20V -> 1uF; footprint Capacitors:0603 -> Capacitor_SMD:C_0603_1608Metric
- C3: value 10uF 20V -> 10uF X5R/X7R 25V; footprint Capacitors:0805 -> Capacitor_SMD:C_0603_1608Metric
- C4: value 10uF 20V -> NC; footprint Capacitors:0805 -> Capacitor_SMD:C_0603_1608Metric
- C5: value 100nF 50V -> NC; footprint Capacitors:0603 -> Capacitor_SMD:C_0603_1608Metric
- C6, C7: value 4.7uF 50V -> 1uF; footprint Capacitors:0603 -> Capacitor_SMD:C_0603_1608Metric
- C8, C9: value 22uF -> 200-600pF; footprint Capacitors:0805 -> Capacitor_SMD:C_0603_1608Metric
- J3: footprint Connector_PinHeader_2.54mm:PinHeader_2x05_P2.54mm_Vertical -> Connector_PinHeader_2.54mm:PinHeader_2x05_P2.54mm_Vertical_SMD
- R1: value 54K9 -> NC; footprint Resistors:0603 -> Resistor_SMD:R_0603_1608Metric
- R3, R4: footprint Resistors:0603 -> Resistor_SMD:R_0603_1608Metric
- R5: value 22K -> 1K; footprint Resistors:0603 -> Resistor_SMD:R_0603_1608Metric
- R6: value 5K -> 1K; footprint Resistors:0603 -> Resistor_SMD:R_0603_1608Metric
- R7: value 22.1K -> NC
- R8: value 47.5K -> 0
- TP1, TP2: footprint Connectors:PAD.03X.03 -> digikey-footprints:Test-Point-Pin_Drill2.79mm
- TP3, TP4: footprint Connectors:PAD.03X.03 -> TestPoint:TestPoint_Pad_D1.5mm
Connections:
- net 5V: now also TP1.1, C24.1, C25.1, C26.1, C27.1, C28.1, C29.2, C30.2, L7.1, L7.2, R13.2, R16.1, U4.7 (VOUT), U4.8 (VOUT), U5.7 (REGIN); no longer C10.2, C15.1, C16.1, C8.2, C9.2, R1.1
- net CC1: now also C9.1, C21.1, J5.A5 (CC1), U1.5 (IO4), U1.6 (NC), U2.1 (CC1DB), U2.2 (CC1), U3.4 (IO3), U3.7 (NC); no longer C11.1
- net CC2: now also C8.1, C22.1, J5.B5 (CC2), U1.1 (IO1), U1.10 (NC), U2.4 (CC2), U2.5 (CC2DB), U3.5 (IO4), U3.6 (NC); no longer C12.1
- net D+: now also FL1.1, FL2.1, J5.A7 (D-), J5.B7 (D-), R19.2
- net D-: now also FL1.3, FL2.3, J5.A6 (D+), J5.B6 (D+), R18.2
- net GND: now also C10.2, C13.1, C16.1, C2.2, C3.2, C4.2, C5.2, C6.2, C8.2, C9.2, C1.2, C19.2, C20.2, C21.2, C22.2, C23.2, C24.2, C25.2, C26.2, C27.2, C28.2, C29.1, C30.1, C31.1, C32.1, C33.1, D3.2 (A), FL3.4, J5.A1 (GND), J5.A12 (GND), J5.B1 (GND), J5.B12 (GND), R11.2, R14.1, R17.2, U1.3 (G), U1.8 (G), U2.10 (GND), U2.12 (ADDR0), U2.13 (ADDR1), U2.25 (GND), U2.6 (RESET), U3.3 (G), U3.8 (G), U4.10 (NCGND), U4.11 (NCGND), U4.15 (PGND), U4.3 (NCGND), U5.2 (GND), U5.25 (GND); no longer C10.1, C13.2, C14.2, C16.2, C2.1, C3.1, C4.1, C6.1, C8.1, C9.1, J1.A1 (GND), J1.A12 (GND), J1.B1 (GND), J1.B12 (GND), J1.S1 (SHIELD), R3.2, R6.2, R8.2
- net SCL: now also U2.7 (SCL)
- net SDA: now also U2.8 (SDA)
- net VBUS: now also C6.1, R1.1, R3.1, R5.2, Q1.1 (S), Q1.2 (S), Q1.3 (S), R10.2, R22.2, U2.24 (VDD); no longer C6.2, J1.A4 (VBUS), J1.A9 (VBUS), J1.B4 (VBUS), J1.B9 (VBUS)
- net at R1.2: now also C1.1
- net at C5.1: now also FL1.4, U1.2 (IO2), U1.9 (NC)
- net VBUSOK: now reaches R4.1
- net VBUSOK: now also C10.1, C11.1, C12.1, C14.1, C3.1, R8.1, TP2.1, C23.1, L3.1, L3.2, Q1.5_6_7_8 (D), U4.1 (VIN), U4.14 (VIN)
- net at C17.1: now also FL2.4, U3.1 (IO1), U3.10 (NC); no longer C18.1
- net at R7.2: now also C15.1; no longer R8.1
- net at J1.A2 (TX1+): no longer TP4.1
- net at J1.A3 (TX1-): no longer TP3.1
- net at J1.B10 (RX1-): no longer TP1.1
- net at J1.B11 (RX1+): no longer TP2.1
- net BAT_SENSE: no longer names the net of R6.1
- net BAT_SENSE: now also U2.16 (VBUS_EN_SNK); no longer R5.2
- net CHARGE_STAT: no longer names the net of R4.2
- net CHARGE_STAT: now also U2.9 (DISCH)
- removed net VBAT: C2.2, C3.2, C4.2, C7.2, R5.1
- new net: D1.1 (K), FL3.2, J1.A4 (VBUS), J1.A9 (VBUS), J1.B4 (VBUS), J1.B9 (VBUS)
- new net: Q1.4 (G), R12.1, R5.1, R6.2
- new net: C14.2, R12.2
- new net: D3.1 (K), FB1.2, J5.A4 (VBUS), J5.A9 (VBUS), J5.B4 (VBUS), J5.B9 (VBUS), L1.2
- new net: C20.1, J5.S1 (SHIELD), R11.1
- new net: R3.2, U2.18 (VBUS_VS_DISCH)
- new net: C13.2, U2.23 (VREG_2V7)
- new net: C7.2, U2.21 (VREG_1V2)
- new net: TP3.1, U4.13 (V5V)
- new net: R8.2, U4.2 (EN)
- new net: TP4.1, U4.6 (PGOOD)
- new net: R13.1, R14.2, U4.9 (FB)
- new net: C2.1, FB1.1, L1.1, R10.1
- new net: C16.2, C19.1, FL3.3, R22.1
- new net: C4.1, FL1.2, U1.4 (IO3), U1.7 (NC)
- new net: C18.1, FL2.2, U3.2 (IO2), U3.9 (NC)
- new net: C31.2, C32.2, R21.1, U5.6 (VDD)
- new net: C33.2, R20.1, R21.2, U5.5 (VIO)
- new net: R20.2, U5.9 (~RSTb)
- new net: R16.2, R17.1, U5.8 (VBUS)
- new net: J2.12 (Pin_12), U5.1 (RI/CLK)
- new net: J2.5 (Pin_5), U5.11 (GPIO.3)
- new net: J2.7 (Pin_7), U5.12 (GPIO.2)
- new net: J2.9 (Pin_9), U5.13 (GPIO.1)
- new net: J2.11 (Pin_11), U5.14 (GPIO.0)
- new net: J2.10 (Pin_10), U5.18 (CTS)
- new net: J2.8 (Pin_8), U5.19 (RTS)
- new net: J2.6 (Pin_6), U5.20 (RXD)
- new net: J2.4 (Pin_4), U5.21 (TXD)
- new net: J2.2 (Pin_2), U5.22 (DSR)
- new net: J2.1 (Pin_1), U5.23 (DTR)
- new net: J2.3 (Pin_3), U5.24 (DCD)
- new net: R18.1, U5.3 (D+)
- new net: R19.1, U5.4 (D-)
- new net ALERT: U2.19 (ALERT)
- new net ATTACH: U2.11 (ATTACH)
- new net A_B_SIDE: U2.17 (A_B_SIDE)
- new net GPIO: U2.15 (GPIO)
- new net POER_OK2: U2.20 (POWER_OK2)
- new net POER_OK3: U2.14 (POWER_OK3)
- new net S1: D1.2 (A), FL3.1, J1.A1 (GND), J1.A12 (GND), J1.B1 (GND), J1.B12 (GND), J1.S1 (SHIELD)
- no-connect marks 9 -> 10
Other:
- note removed: "VBUS PD TO 9V"
- moved on the sheet: J1, J3, TP12, TP13

Commit message: m
Parts:
- removed C22: 200-600pF, Capacitor_SMD:C_0603_1608Metric, symbol Device:C
- removed FL1, FL2: 0603USB-251MLB, Inductor_SMD:L_CommonModeChoke_Coilcraft_0603USB, symbol Device:EMI_Filter_CommonMode
- removed TP3, TP4: TestPoint, TestPoint:TestPoint_Pad_D1.5mm, symbol Connector:TestPoint
- removed U3: TPD4E02B04DQA, aep:USON-10_2.5x1.0mm_P0.5mm_HAXED_MIDDLE, symbol aep:TPD4E02B04DQA
- added D10, D2, D4, D5, D6, D7, D8, D9: LED, digikey-footprints:LED_0603, symbol Device:LED
- added FL1: 0603USB-251MLB, Inductor_SMD:L_CommonModeChoke_Coilcraft_0603USB, symbol aep:EMI_Filter_CommonMode_1243
- added J10, J11, J12, J4, J6, J7, J8, J9: Conn_01x04_Female, aep:Castellated_Edge_1x4_P2.54mm, symbol Connector:Conn_01x04_Female
- added J13: Conn_01x06, Connector:Tag-Connect_TC2030-IDC-FP_2x03_P1.27mm_Vertical, symbol Connector_Generic:Conn_01x06
- added R15, R2, R23, R24, R25, R27, R9: 1K, Resistor_SMD:R_0603_1608Metric, symbol Device:R
- added R26: 100K, Resistor_SMD:R_0603_1608Metric, symbol Device:R
- added U3: STM32F070F6Px, Package_SO:TSSOP-20_4.4x6.5mm_P0.65mm, symbol MCU_ST_STM32F0:STM32F070F6Px
- added U6: AZ1117CH-3_3TRG1, digikey-footprints:SOT-223, symbol dk_PMIC-Voltage-Regulators-Linear:AZ1117CH-3_3TRG1
- C15, C17, C18: value NC -> 10uF
- C21: value 200-600pF -> 10uF
- R22: value 0 -> 1K
- R7: value NC -> 1K
Connections:
- net INT is gone; now on net SCL: J3.5 (Pin_5)
- net RTS is gone; now on net ATTACH: J3.8 (Pin_8)
- net RXD is gone; now on net POER_OK2: J3.7 (Pin_7)
- net TXD is gone; now on net POER_OK3: J3.6 (Pin_6)
- net 5V: now also C15.1, D9.2 (A), J10.1 (Pin_1), J10.2 (Pin_2), J10.3 (Pin_3), J10.4 (Pin_4), J9.1 (Pin_1), J9.2 (Pin_2), J9.3 (Pin_3), J9.4 (Pin_4), U6.3 (IN)
- net ALERT: now also J3.2 (Pin_2), R22.2
- net ATTACH: now also R9.2
- net A_B_SIDE: now also J3.3 (Pin_3), R23.2
- net CC1: no longer C21.1
- net D+: now also C4.1, FL1.3, U3.18 (PA10/PA12); no longer J1.A7 (D-), J1.B7 (D-), J5.A7 (D-), J5.B7 (D-)
- net D-: now also C5.1, FL1.2, U3.17 (PA9/PA11); no longer J1.A6 (D+), J1.B6 (D+), J5.A6 (D+), J5.B6 (D+)
- net GND: now also FL3.3, U4.12 (AGND), J11.1 (Pin_1), J11.2 (Pin_2), J11.3 (Pin_3), J11.4 (Pin_4), J12.1 (Pin_1), J12.2 (Pin_2), J12.3 (Pin_3), J12.4 (Pin_4), J13.5 (Pin_5), J4.1 (Pin_1), J4.2 (Pin_2), J4.3 (Pin_3), J4.4 (Pin_4), J6.1 (Pin_1), J6.2 (Pin_2), J6.3 (Pin_3), J6.4 (Pin_4), J7.1 (Pin_1), J7.2 (Pin_2), J7.3 (Pin_3), J7.4 (Pin_4), J8.1 (Pin_1), J8.2 (Pin_2), J8.3 (Pin_3), J8.4 (Pin_4), R15.2, R24.2, R27.2, U3.15 (VSS), U6.1 (ADJ/GND); no longer FL3.4, U1.3 (G), U1.8 (G)
- net POER_OK2: now also R7.2
- net POER_OK3: now also R2.2
- net S1: now also FL3.2, U1.3 (G), U1.8 (G); no longer FL3.1
- net SCL: no longer J3.4 (Pin_4)
- net SDA: now also J3.4 (Pin_4); no longer J3.3 (Pin_3)
- net VBUS: now also C16.2, C19.1, FL3.4; no longer R22.2, R7.1
- net VIN: now reaches D1.1 (K), J1.A4 (VBUS), J1.A9 (VBUS), J1.B4 (VBUS), J1.B9 (VBUS)
- net VIN: now also FL3.1; no longer FL3.2
- net STUSB_VSYS: now reaches J3.1 (Pin_1)
- net STUSB_VSYS: now also U2.22 (VSYS), D2.2 (A), D4.2 (A), D5.2 (A), D6.2 (A), D7.2 (A), D8.2 (A)
- net at U4.13 (V5V): now also D10.2 (A), R26.1
- net at U4.6 (PGOOD): now also R25.2, R26.2
- net IN_D+: now reaches U1.2 (IO2), U1.9 (NC)
- net IN_D+: now also J1.A7 (D-), J1.B7 (D-), J5.A7 (D-), J5.B7 (D-), FL1.1; no longer C5.1
- net IN_D-: now reaches U1.4 (IO3), U1.7 (NC)
- net IN_D-: now also J1.A6 (D+), J1.B6 (D+), J5.A6 (D+), J5.B6 (D+), FL1.4; no longer C4.1
- net 3.3V: now reaches C17.1
- net 3.3V: now also C18.1, C21.1, J13.1 (Pin_1), U3.16 (VDD), U3.5 (VDDA), U6.2 (OUT), U6.4 (VOUT)
- net USART_RTS: now reaches J2.8 (Pin_8), U5.19 (RTS)
- net USART_RTS: now also U3.7 (PA1)
- net USART_RX: now reaches J2.6 (Pin_6), U5.20 (RXD)
- net USART_RX: now also U3.9 (PA3)
- net USART_TX: now reaches J2.4 (Pin_4), U5.21 (TXD)
- net USART_TX: now also U3.8 (PA2)
- net USART_DTR: now reaches J2.1 (Pin_1), U5.23 (DTR)
- net USART_DTR: now also U3.10 (PA4)
- net CTS: no longer names the net of J3.9 (Pin_9)
- new net: R27.1, U3.1 (BOOT0)
- new net: D8.1 (K), R23.1
- new net: D7.1 (K), R22.1
- new net: D6.1 (K), R15.1
- new net: D5.1 (K), R9.1
- new net: D4.1 (K), R7.1
- new net: D2.1 (K), R2.1
- new net: D9.1 (K), R24.1
- new net: D10.1 (K), R25.1
- new net USART_RESET: J13.3 (Pin_3), U3.4 (NRST)
- new net USART_SWD_CLK: J13.4 (Pin_4), U3.20 (PA14)
- new net USART_SWD_IO: J13.2 (Pin_2), U3.19 (PA13)
- no-connect marks 10 -> 14
Other:
- moved on the sheet: C23, C4, C5, C8, C9, U1
